Commit message: Simulation Completed Project

File: description/depth_camera.xacro (robot description, xacro)
@@ -29,5 +29,6 @@
                 <horizontal_fov>1.089</horizontal_fov>
                 <image>
-                    <format>R8G8B8</format>
+                    <!-- <format>R8G8B8</format>  -->
+                    <format>B8G8R8</format>
                     <width>640</width> <!-- horizontal resolution -->
                     <height>480</height> <!-- vertical resolution -->

File: description/lidar.xacro (robot description, xacro)
@@ -1,4 +1,2 @@
-<!--                          UNUSED                       -->
-<?xml version="1.0"?>
 <robot xmlns:xacro="http://www.ros.org/wiki/xacro" >
     <joint name="laser_joint" type="fixed">

File: description/lidar_3d.xacro (robot description, xacro)
@@ -11,18 +11,20 @@
                 <cylinder radius="0.05" length="0.04"/> <!-- little cylinder -->
             </geometry>
-            <material name="orange"/>
+            <material name="black"/>
         </visual>
-        <collision> <!-- physic collision -->
+        <!--
+        <collision>  physic collision
             <geometry>
-                <cylinder radius="0.05" length="0.04"/> <!-- same shape-->
+                <cylinder radius="0.05" length="0.04"/>  same shape
             </geometry>
         </collision>
-        <xacro:inertial_cylinder mass="0.1" length="0.04" radius="0.05">
+        -->
+        <xacro:inertial_cylinder mass="0.0" length="0.04" radius="0.05">
             <origin xyz="0 0 0" rpy="0 0 0"/>
         </xacro:inertial_cylinder>
     </link>
     <!-- gazebo definitions-->
-    <gazebo reference="laser_frame">
-        <material>Gazebo/Orange</material>
+    <gazebo reference="laser_frame" collision="false">
+        <material>Gazebo/Black</material>
         <!-- LIDAR sensor (ray) -->
         <sensor name="laser" type="ray">

File: description/robot.urdf.xacro (robot description, xacro)
@@ -10,5 +10,8 @@
         <xacro:include filename="gazebo_control.xacro" />
     </xacro:unless>
-    <xacro:if value="${'$(arg sensors)' == 'lidar_3D'}">
+    <xacro:if value="${'$(arg sensors)' == 'lidar'}">
+        <xacro:include filename="lidar.xacro" />
+    </xacro:if>
+    <xacro:if value="${'$(arg sensors)' == 'lidar_3D' or '$(arg sensors)' == 'lidar_3D_and_Slam'}">
         <xacro:include filename="lidar_3d.xacro" />
         <xacro:include filename="camera.xacro" />

File: description/robot_core.xacro (robot description, xacro)
@@ -24,4 +24,12 @@
     <!-- BASE LINK -->
     <link name="base_link"> <!-- main reference for all the other links -->
+    </link>
+    <!-- BASE_FOOTPRINT LINK -->
+    <joint name="base_footprint_joint" type="fixed">
+        <parent link="base_link"/>
+        <child link="base_footprint"/>
+        <origin xyz="0 0 0" rpy="0 0 0"/>
+    </joint>
+    <link name="base_footprint">
     </link>
     <!-- CHASSIS LINK -->
